Commit message: registered workspace, enable communication with matlab, move to single point from terminal input

File: src/irb120_description/urdf/abb_irb120(DH).urdf (robot description, URDF)
Before this commit: robot abb_irb120, 10 links, 9 joints
Joints:
- joint joint6-end_effector: origin xyz=0.082 0 0 rpy=0 0 0 -> xyz=0 0 0.082 rpy=0 0 0
- joint joint_1: origin xyz=0 0 0 rpy=0 0 0 -> xyz=0 0 0.187 rpy=0 0 0
- joint joint_2: axis 0 1 0 -> 0 0 1; origin xyz=0 0 0.29 rpy=0 0 0 -> xyz=0 0 0.103 rpy=-1.57079632679 0 0
- joint joint_3: axis 0 1 0 -> 0 0 1; origin xyz=0 0 0.27 rpy=0 0 0 -> xyz=0 -0.27 0 rpy=0 0 0
- joint joint_4: axis 1 0 0 -> 0 0 1; origin xyz=0 0 0.07 rpy=0 0 0 -> xyz=0 -0.07 0 rpy=0 1.57079632679 0
- joint joint_5: axis 0 1 0 -> 0 0 1; origin xyz=0.302 0 0 rpy=0 0 0 -> xyz=0 0 0.302 rpy=0 -1.57079632679 0
- joint joint_6: axis 1 0 0 -> 0 0 1; origin xyz=0.072 0 0 rpy=0 0 0 -> xyz=0.072 0 0 rpy=0 1.57079632679 0
